Commit message: feat(phase-3): deterministic waypoint_follower replaces Nav2 for driving (simple+stable)
Retest plan change (user-approved, roadmap updated first). The gravity-free planar abstraction with ground-truth odometry made Nav2's reactive stack the sole source of path-following instability (corner-cut, phantom obstacle, in-place spin). Switched the default driving controller to a deterministic turn-then-drive node; Nav2 retained as documented advanced mode.

- window_cleaner_planning/waypoint_follower.py (new): consumes /planning/coverage_path + ground-truth /odom, applies static spawn frame_offset, publishes /cmd_vel and /control/mission_state (downstream contract preserved). Verified end-to-end: RUNNING -> DONE, clean turn-drive-turn.

- coverage_planner.py: latched /planning/glass_boundary_viz (window rectangle) for Foxglove (no Nav2 /map in simple mode).

- sim.launch.py: static map->odom TF, arg map_odom_tf (default true; set false for Nav2 mode).

- robot.urdf.xacro: drop camera_link <visual>+<collision> — gpu_lidar renders visuals, self-detected the camera box ~0.11 m ahead -> permanent phantom obstacle/RPP abort.

- nav2.launch.py + config/bt/navigate_through_poses_coverage.xml (new): custom NavigateThroughPoses BT, RemovePassedGoals radius 0.15 (default 0.7 > strip spacing 0.2875 -> corner-cut). Advanced Nav2 mode.

- setup.py: waypoint_follower entry point. docs/RUNNING.md + RUNNING.tr.md: default=simple, Nav2=advanced. PROJECT_ROADMAP: Phase 3 AI Notes plan-change record.

Co-Authored-By: Claude Opus 4.7 (1M context) <noreply@anthropic.com>

File: src/window_cleaner_description/urdf/robot.urdf.xacro (robot description, xacro)
@@ -112,13 +112,20 @@
   <xacro:wheel prefix="rear_right"  x_sign="-1" y_sign="-1"/>
   <link name="camera_link">
-    <visual>
-      <origin xyz="0 0 0"/>
-      <geometry><box size="${camera_size} ${camera_size} ${camera_size}"/></geometry>
-      <material name="camera_red"/>
-    </visual>
-    <collision>
-      <origin xyz="0 0 0"/>
-      <geometry><box size="${camera_size} ${camera_size} ${camera_size}"/></geometry>
-    </collision>
+    <!-- No <visual> and no <collision> on purpose.
+         The frame walls are only 0.10 m tall (world z in [0.005, 0.105]),
+         but this robot is taller: with spawn z=0.05 the lidar scan plane
+         sits at world z=0.155, ABOVE the walls, so the 360 gpu_lidar never
+         sees the frame at all. gpu_lidar is GPU-render based -> it detects
+         VISUAL geometry, not collision. The camera housing's visual box
+         spans world z in [0.14, 0.18] and x in [0.11, 0.15] (forward of
+         base centre), i.e. exactly across the lidar plane ~0.11 m dead
+         ahead. The lidar therefore self-detected the camera box as a
+         permanent obstacle and RPP aborted every mission with
+         "collision ahead -> patience exceeded" (removing only <collision>
+         did nothing because gpu_lidar ignores collision). Dropping the
+         visual makes the camera invisible to the lidar render pass; the
+         rgb_camera sensor (attached via <gazebo reference="camera_link">)
+         and the link inertia are unaffected. Real frame avoidance comes
+         from the static map in the global costmap, not this lidar. -->
     <xacro:box_inertia m="${camera_mass}" x="${camera_size}" y="${camera_size}" z="${camera_size}"/>
   </link>
